Commit message: Changed the ur communication to sockets instead of topics

File: src/ur_robot/universal_robot/universal_robot/ur_description/urdf/ur10.urdf.xacro (robot description, xacro)
@@ -280,5 +280,5 @@
                  degrees)
       -->
-      <origin xyz="0 0 0" rpy="0 0 ${-pi}"/>
+      <origin xyz="0 0 0" rpy="0 0 0"/>
       <parent link="${prefix}base_link"/>
       <child link="${prefix}base"/>

File: src/ur_robot/universal_robot/universal_robot/ur_description/urdf/ur10_robot.urdf.xacro (robot description, xacro)
@@ -12,5 +12,5 @@
     <parent link="world" />
     <child link = "base_link" />
-    <origin xyz="0.0 0.0 0.0" rpy="0.0 0.0 0.0" />
+    <origin xyz="0.0 0.0 0.3" rpy="0.0 0.0 0.0" />
   </joint>
 </robot>
